File: PCB/SCHEMATIC/CNC BATTERY/SCHEMATIC/SPARC CNC with battery.brd (EAGLE design)
At the start: 70 x 40 mm, 12 parts

Commit message: Update
Parts:
- removed MP: MP1584, MP1584-dc-brick (1):DC-BRICK
- added OUT+, OUT-, VIN+, VIN-: (no value), pinhead:1X02
- moved BATTERY 2.81 mm to (13.2, 36.3)
Connections:
- net +: now also VIN+.1, VIN+.2; no longer MP.IN1+, MP.IN2+
- net -: now also VIN-.1, VIN-.2; no longer MP.IN1-, MP.IN2-
- net OUT+: now also OUT+.1, OUT+.2; no longer MP.OUT1+, MP.OUT2+
- net OUT-: now also OUT-.1, OUT-.2; no longer MP.OUT1-, MP.OUT2-
Routing:
- net +: track 75.7 -> 72.6 mm
- net B-: track 44.2 -> 47.3 mm
- net B+: track 63.6 -> 66.0 mm
- net OUT+: track 93.4 -> 91.5 mm
- net OUT-: track 44.4 -> 45.9 mm
- net PIN33: track 54.7 -> 55.3 mm
- net -: track 121.7 -> 122.3 mm
- added copper zone on layer 15, net 0V
- removed copper zone on layer 15, net GND
Other:
- board text added: "+"
- board text added: "-"
- board text added: "10K"
- board text added: "22K"
- board text added: "3K3"
- board text added: "ANODA"
- board text added: "CATHODA"
- board text added: "D"
- board text added: "G"
- board text added: "S"
- board text added: "SIG"
