File: PCB/SCHEMATIC/CNC BATTERY/SCHEMATIC/SPARC CNC with battery.sch (EAGLE design)
At the start: 12 parts

Commit message: Update
Parts:
- removed MP: MP1584, MP1584-dc-brick (1):MP1584
- added OUT+, OUT-, VIN+, VIN-: (no value), pinhead:PINHD-1X2
Connections:
- net +: now also VIN+.1, VIN+.2; no longer MP.VIN+
- net -: now also VIN-.1, VIN-.2; no longer MP.VIN-
- net OUT+: now also OUT+.1, OUT+.2; no longer MP.VOUT+
- net OUT-: now also OUT-.1, OUT-.2; no longer MP.VOUT-
Changed lines of the file:
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@@
 </classes>
 <parts>
-<part name="MP" library="MP1584-dc-brick (1)" deviceset="MP1584" device=""/>
 <part name="TP" library="32teeth - TP4056 Module" deviceset="TP4056-PTH" device=""/>
 <part name="BATTERY" library="pinhead-2" deviceset="PINHD-1X02" device="_2.54"/>
@@
 <part name="LED2" library="pinhead" library_urn="urn:adsk.eagle:library:325" deviceset="PINHD-1X2" device="" package3d_urn="urn:adsk.eagle:package:22435/2"/>
 <part name="INPUT" library="pinhead" library_urn="urn:adsk.eagle:library:325" deviceset="PINHD-1X2" device="" package3d_urn="urn:adsk.eagle:package:22435/2"/>
+<part name="VIN+" library="pinhead" library_urn="urn:adsk.eagle:library:325" deviceset="PINHD-1X2" device="" package3d_urn="urn:adsk.eagle:package:22435/2"/>
+<part name="VIN-" library="pinhead" library_urn="urn:adsk.eagle:library:325" deviceset="PINHD-1X2" device="" package3d_urn="urn:adsk.eagle:package:22435/2"/>
+<part name="OUT+" library="pinhead" library_urn="urn:adsk.eagle:library:325" deviceset="PINHD-1X2" device="" package3d_urn="urn:adsk.eagle:package:22435/2"/>
+<part name="OUT-" library="pinhead" library_urn="urn:adsk.eagle:library:325" deviceset="PINHD-1X2" device="" package3d_urn="urn:adsk.eagle:package:22435/2"/>
 </parts>
 <sheets>
@@
 </plain>
 <instances>
-<instance part="MP" gate="G$1" x="119.38" y="86.36" smashed="yes"/>
 <instance part="TP" gate="G$1" x="172.72" y="86.36" smashed="yes"/>
 <instance part="BATTERY" gate="A" x="218.44" y="86.36" smashed="yes">
@@
 <attribute name="VALUE" x="113.03" y="104.14" size="1.778" layer="96"/>
 </instance>
+<instance part="VIN+" gate="G$1" x="76.2" y="101.6" smashed="yes">
+<attribute name="NAME" x="69.85" y="107.315" size="1.778" layer="95"/>
+<attribute name="VALUE" x="69.85" y="96.52" size="1.778" layer="96"/>
+</instance>
+<instance part="VIN-" gate="G$1" x="76.2" y="83.82" smashed="yes">
+<attribute name="NAME" x="69.85" y="89.535" size="1.778" layer="95"/>
+<attribute name="VALUE" x="69.85" y="78.74" size="1.778" layer="96"/>
+</instance>
+<instance part="OUT+" gate="G$1" x="93.98" y="101.6" smashed="yes">
+<attribute name="NAME" x="87.63" y="107.315" size="1.778" layer="95"/>
+<attribute name="VALUE" x="87.63" y="96.52" size="1.778" layer="96"/>
+</instance>
+<instance part="OUT-" gate="G$1" x="93.98" y="83.82" smashed="yes">
+<attribute name="NAME" x="87.63" y="89.535" size="1.778" layer="95"/>
+<attribute name="VALUE" x="87.63" y="78.74" size="1.778" layer="96"/>
+</instance>
 </instances>
 <busses>
@@
 <nets>
 <net name="OUT+" class="0">
-<segment>
-<pinref part="MP" gate="G$1" pin="VOUT+"/>
-<wire x1="137.16" y1="88.9" x2="142.24" y2="88.9" width="0.1524" layer="91"/>
-<label x="144.78" y="86.36" size="1.778" layer="95" rot="R90"/>
-</segment>
 <segment>
 <pinref part="TP" gate="G$1" pin="IN+"/>
@@
 <pinref part="DIODA" gate="G$1" pin="A"/>
 </segment>
+<segment>
+<pinref part="OUT+" gate="G$1" pin="2"/>
+<wire x1="91.44" y1="101.6" x2="86.36" y2="101.6" width="0.1524" layer="91"/>
+<label x="83.82" y="99.06" size="1.778" layer="95" rot="R90"/>
+<pinref part="OUT+" gate="G$1" pin="1"/>
+<wire x1="91.44" y1="104.14" x2="86.36" y2="104.14" width="0.1524" layer="91"/>
+<wire x1="91.44" y1="104.14" x2="91.44" y2="101.6" width="0.1524" layer="91"/>
+<junction x="91.44" y="104.14"/>
+<junction x="91.44" y="101.6"/>
+</segment>
 </net>
 <net name="B+" class="0">
@@
 <net name="OUT-" class="0">
 <segment>
-<pinref part="MP" gate="G$1" pin="VOUT-"/>
-<wire x1="137.16" y1="83.82" x2="142.24" y2="83.82" width="0.1524" layer="91"/>
-<label x="142.24" y="83.82" size="1.778" layer="95" rot="R270"/>
-</segment>
-<segment>
 <pinref part="TP" gate="G$1" pin="IN-"/>
 <wire x1="162.56" y1="83.82" x2="160.02" y2="83.82" width="0.1524" layer="91"/>
 <label x="154.94" y="83.82" size="1.778" layer="95"/>
 </segment>
+<segment>
+<pinref part="OUT-" gate="G$1" pin="2"/>
+<wire x1="91.44" y1="83.82" x2="86.36" y2="83.82" width="0.1524" layer="91"/>
+<label x="86.36" y="81.28" size="1.778" layer="95" rot="R270"/>
+<pinref part="OUT-" gate="G$1" pin="1"/>
+<wire x1="91.44" y1="86.36" x2="86.36" y2="86.36" width="0.1524" layer="91"/>
+<wire x1="91.44" y1="86.36" x2="91.44" y2="83.82" width="0.1524" layer="91"/>
+<junction x="91.44" y="86.36"/>
+<junction x="91.44" y="83.82"/>
+</segment>
 </net>
 <net name="+" class="0">
-<segment>
-<pinref part="MP" gate="G$1" pin="VIN+"/>
-<wire x1="104.14" y1="88.9" x2="101.6" y2="88.9" width="0.1524" layer="91"/>
-<label x="101.6" y="88.9" size="1.778" layer="95" rot="R180"/>
-</segment>
 <segment>
 <pinref part="R1" gate="G$1" pin="1"/>
@@
 <wire x1="116.84" y1="109.22" x2="114.3" y2="109.22" width="0.1524" layer="91"/>
 <label x="111.76" y="109.22" size="1.778" layer="95"/>
+</segment>
+<segment>
+<pinref part="VIN+" gate="G$1" pin="2"/>
+<wire x1="73.66" y1="101.6" x2="66.04" y2="101.6" width="0.1524" layer="91"/>
+<label x="66.04" y="101.6" size="1.778" layer="95"/>
+<pinref part="VIN+" gate="G$1" pin="1"/>
+<wire x1="73.66" y1="104.14" x2="66.04" y2="104.14" width="0.1524" layer="91"/>
+<wire x1="73.66" y1="104.14" x2="73.66" y2="101.6" width="0.1524" layer="91"/>
+<junction x="73.66" y="104.14"/>
+<junction x="73.66" y="101.6"/>
 </segment>
 </net>
@@
 <net name="-" class="0">
 <segment>
-<pinref part="MP" gate="G$1" pin="VIN-"/>
-<wire x1="104.14" y1="83.82" x2="101.6" y2="83.82" width="0.1524" layer="91"/>
-<label x="101.6" y="83.82" size="1.778" layer="95" rot="R180"/>
-</segment>
-<segment>
 <pinref part="INPUT" gate="G$1" pin="1"/>
 <wire x1="116.84" y1="111.76" x2="114.3" y2="111.76" width="0.1524" layer="91"/>
@@
 <label x="149.86" y="27.94" size="1.778" layer="95"/>
 </segment>
+<segment>
+<pinref part="VIN-" gate="G$1" pin="2"/>
+<wire x1="73.66" y1="83.82" x2="66.04" y2="83.82" width="0.1524" layer="91"/>
+<label x="63.5" y="83.82" size="1.778" layer="95"/>
+<pinref part="VIN-" gate="G$1" pin="1"/>
+<wire x1="73.66" y1="86.36" x2="66.04" y2="86.36" width="0.1524" layer="91"/>
+<wire x1="73.66" y1="86.36" x2="73.66" y2="83.82" width="0.1524" layer="91"/>
+<junction x="73.66" y="86.36"/>
+<junction x="73.66" y="83.82"/>
+</segment>
 </net>
